Commit message: modified:   compose.yml 	modified:   docker/Dockerfile 	modified:   scripts/pi_bringup.sh 	new file:   src/mekk4_bringup/mekk4_bringup/bno085_node.py 	modified:   src/mekk4_bringup/package.xml 	modified:   src/mekk4_bringup/setup.py 	modified:   src/robot_bringup/launch/pi_robot.launch.py 	modified:   src/robot_bringup/package.xml 	modified:   src/robot_description/urdf/two_wheel_robot.urdf

File: src/robot_description/urdf/two_wheel_robot.urdf (robot description, URDF)
Before this commit: robot two_wheel_robot, 7 links, 6 joints
Links:
- added link imu_link; visual box size=0.03 0.02 0.01
Joints:
- added joint imu_joint: type fixed, parent chassis, child imu_link, origin xyz=0 0 0.04 rpy=0 0 0

Commit message: modified:   src/robot_bringup/package.xml 	modified:   src/robot_description/urdf/two_wheel_robot.urdf 	modified:   src/robot_gz/worlds/robot3.sdf

File: src/robot_description/urdf/two_wheel_robot.urdf (robot description, URDF)
Before this commit: robot two_wheel_robot, 7 links, 6 joints
Joints:
- joint lidar_joint: origin xyz=0 0 0.13 rpy=0 0 0 -> xyz=0 0 0.18 rpy=0 0 0

Commit message: modified:   src/robot_bringup/launch/lidar_nav2_compat.launch.py 	modified:   src/robot_bringup/launch/minimal_all.launch.py 	modified:   src/robot_bringup/launch/pi_robot.launch.py 	modified:   src/robot_description/urdf/two_wheel_robot.urdf 	modified:   src/robot_gz/worlds/robot3.sdf

File: src/robot_description/urdf/two_wheel_robot.urdf (robot description, URDF)
Before this commit: robot two_wheel_robot, 7 links, 6 joints
Links:
- link caster_wheel: geometry collision sphere radius=0.04
- link chassis: geometry collision box size=0.4 0.3 0.15; visual box size=0.34 0.08 0.14
