Commit message: modified:   src/robot_bringup/launch/minimal_all.launch.py 	modified:   src/robot_bringup/launch/pi_robot.launch.py 	renamed:    src/robot_description/urdf/two_wheel_robot.urdf -> src/robot_description/urdf/tracked_robot.urdf 	renamed:    src/robot_gz/worlds/robot3.sdf -> src/robot_gz/worlds/tracked_robot_world.sdf

File: src/robot_description/urdf/tracked_robot.urdf (robot description, URDF)
Before this commit: robot two_wheel_robot, 7 links, 6 joints
Links:
- link camera_link: geometry visual box size=0.04 0.05 0.03
- link chassis: geometry collision box size=0.297 0.21 0.085; visual box size=0.19 0.038 0.09
- link left_wheel: geometry collision cylinder length=0.03 radius=0.05
- link lidar_link: geometry visual cylinder length=0.04 radius=0.035
- link right_wheel: geometry collision cylinder length=0.03 radius=0.05
Joints:
- joint camera_joint: origin xyz=0.2 0 0.05 rpy=0 0 0 -> xyz=0.125 0 0.06 rpy=0 0 0
- joint caster_joint: origin xyz=0.15 0 -0.10 rpy=0 0 0 -> xyz=0.11 0 -0.07 rpy=0 0 0
- joint imu_joint: origin xyz=0 0 0.04 rpy=0 0 0 -> xyz=0 0 0.03 rpy=0 0 0
- joint left_wheel_joint: origin xyz=-0.1 0.175 -0.06 rpy=-1.5708 0 0 -> xyz=0 0.093 -0.035 rpy=-1.5708 0 0
- joint lidar_joint: origin xyz=0 0 0.18 rpy=0 0 0 -> xyz=0.11 -0.06 0.065 rpy=0 0 0
- joint right_wheel_joint: origin xyz=-0.1 -0.175 -0.06 rpy=-1.5708 0 0 -> xyz=0 -0.093 -0.035 rpy=-1.5708 0 0

Commit message: modified:   src/robot_bringup/CMakeLists.txt 	modified:   src/robot_bringup/launch/minimal_all.launch.py 	modified:   src/robot_bringup/package.xml 	modified:   src/robot_bringup/rviz/minimal_all.rviz 	modified:   src/robot_description/urdf/tracked_robot.urdf 	modified:   src/robot_gz/worlds/tracked_robot_world.sdf 	new file:   src/robot_minimal_control/robot_minimal_control/sim_cmd_vel_calibrator.py 	modified:   src/robot_minimal_control/robot_minimal_control/sim_keyboard_teleop.py 	modified:   src/robot_minimal_control/setup.py

File: src/robot_description/urdf/tracked_robot.urdf (robot description, URDF)
Before this commit: robot tracked_robot, 7 links, 6 joints
Joints:
- joint left_wheel_joint: origin xyz=0 0.093 -0.035 rpy=-1.5708 0 0 -> xyz=-0.035 0.093 -0.02 rpy=-1.5708 0 0
- joint right_wheel_joint: origin xyz=0 -0.093 -0.035 rpy=-1.5708 0 0 -> xyz=-0.035 -0.093 -0.02 rpy=-1.5708 0 0

Commit message: modified:   src/robot_description/urdf/tracked_robot.urdf

File: src/robot_description/urdf/tracked_robot.urdf (robot description, URDF)
Before this commit: robot tracked_robot, 7 links, 6 joints
Joints:
- joint imu_joint: origin xyz=0 0 0.03 rpy=0 0 0 -> xyz=0.11 0 0.03 rpy=0 0 0

Commit message: modified:   src/robot_description/urdf/tracked_robot.urdf

File: src/robot_description/urdf/tracked_robot.urdf (robot description, URDF)
Before this commit: robot tracked_robot, 7 links, 6 joints
Joints:
- joint lidar_joint: origin xyz=0.0 -0.06 0.065 rpy=0 0 0 -> xyz=0.11 0.0 0.065 rpy=0 0 0

Commit message: new file:   AGENTS.md 	modified:   config/ekf.yaml 	modified:   config/nav2_params.yaml 	new file:   frames_2026-04-23_21.14.02.gv 	new file:   frames_2026-04-23_21.14.02.pdf 	modified:   scripts/sim_stop.sh 	modified:   src/robot_bringup/launch/minimal_all.launch.py 	modified:   src/robot_description/CMakeLists.txt 	new file:   src/robot_description/meshes/Camera.stl 	new file:   src/robot_description/meshes/Drive-L.stl 	new file:   src/robot_description/meshes/Drive-R.stl 	new file:   src/robot_description/meshes/IMU.stl 	new file:   src/robot_description/meshes/Lidar.stl 	new file:   src/robot_description/meshes/ML.stl 	new file:   src/robot_description/meshes/MR.stl 	new file:   src/robot_description/meshes/Midsection.stl 	new file:   src/robot_description/meshes/SLOTLBI.stl 	new file:   src/robot_description/meshes/SLOTLFI.stl 	new file:   src/robot_description/meshes/SLOTRBI.stl 	new file:   src/robot_description/meshes/SLOTRFI.stl 	new file:   src/robot_description/meshes/Stepper-1.stl 	new file:   src/robot_description/meshes/Unyaktig-batteri-mockup-v1.stl 	new file:   src/robot_description/meshes/WheelLB.stl 	new file:   src/robot_description/meshes/WheelLF.stl 	new file:   src/robot_description/meshes/WheelLT.stl 	new file:   src/robot_description/meshes/WheelRB.stl 	new file:   src/robot_description/meshes/WheelRF.stl 	new file:   src/robot_description/meshes/WheelRT.stl 	modified:   src/robot_description/urdf/tracked_robot.urdf 	modified:   src/robot_gz/CMakeLists.txt 	modified:   src/robot_gz/worlds/tracked_robot_world.sdf

File: src/robot_description/urdf/tracked_robot.urdf (robot description, URDF)
Before this commit: robot tracked_robot, 7 links, 6 joints
Links:
- removed link caster_wheel
- added link ML, mass 0.1777283215577954; collision mesh filename=package://robot_description/meshes/ML.stl scale=0.001 0.001 0.001; visual mesh filename=package://robot_description/meshes/ML.stl scale=0.001 0.001 0.001
- added link MR, mass 0.1777283215577954; collision mesh filename=package://robot_description/meshes/MR.stl scale=0.001 0.001 0.001; visual mesh filename=package://robot_description/meshes/MR.stl scale=0.001 0.001 0.001
- added link SLOTLBI, mass 0.021811111801316833; collision mesh filename=package://robot_description/meshes/SLOTLBI.stl scale=0.001 0.001 0.001; visual mesh filename=package://robot_description/meshes/SLOTLBI.stl scale=0.001 0.001 0.001
- added link SLOTLFI, mass 0.021811457974470146; collision mesh filename=package://robot_description/meshes/SLOTLFI.stl scale=0.001 0.001 0.001; visual mesh filename=package://robot_description/meshes/SLOTLFI.stl scale=0.001 0.001 0.001
- added link SLOTRBI, mass 0.021811111801316826; collision mesh filename=package://robot_description/meshes/SLOTRBI.stl scale=0.001 0.001 0.001; visual mesh filename=package://robot_description/meshes/SLOTRBI.stl scale=0.001 0.001 0.001
- added link SLOTRFI, mass 0.02181145797447015; collision mesh filename=package://robot_description/meshes/SLOTRFI.stl scale=0.001 0.001 0.001; visual mesh filename=package://robot_description/meshes/SLOTRFI.stl scale=0.001 0.001 0.001
- added link Stepper-1, mass 0.24015056879172078; collision mesh filename=package://robot_description/meshes/Stepper-1.stl scale=0.001 0.001 0.001; visual mesh filename=package://robot_description/meshes/Stepper-1.stl scale=0.001 0.001 0.001
- added link Unyaktig-batteri-mockup-v1, mass 0.43806049485710546; collision mesh filename=package://robot_description/meshes/Unyaktig-batteri-mockup-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 scale=0.001 0.001 0.001; visual mesh filename=package://robot_description/meshes/Unyaktig-batteri-mockup-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 scale=0.001 0.001 0.001
- added link WheelLB, mass 0.01924516490772345; collision mesh filename=package://robot_description/meshes/WheelLB.stl scale=0.001 0.001 0.001; visual mesh filename=package://robot_description/meshes/WheelLB.stl scale=0.001 0.001 0.001
- added link WheelLF, mass 0.01924516490772345; collision mesh filename=package://robot_description/meshes/WheelLF.stl scale=0.001 0.001 0.001; visual mesh filename=package://robot_description/meshes/WheelLF.stl scale=0.001 0.001 0.001
- added link WheelLT, mass 0.01924516490772345; collision mesh filename=package://robot_description/meshes/WheelLT.stl scale=0.001 0.001 0.001; visual mesh filename=package://robot_description/meshes/WheelLT.stl scale=0.001 0.001 0.001
- added link WheelRB, mass 0.14253267377489354; collision mesh filename=package://robot_description/meshes/WheelRB.stl scale=0.001 0.001 0.001; visual mesh filename=package://robot_description/meshes/WheelRB.stl scale=0.001 0.001 0.001
- added link WheelRF, mass 0.14253267377489354; collision mesh filename=package://robot_description/meshes/WheelRF.stl scale=0.001 0.001 0.001; visual mesh filename=package://robot_description/meshes/WheelRF.stl scale=0.001 0.001 0.001
- added link WheelRT, mass 0.01924645021673722; collision mesh filename=package://robot_description/meshes/WheelRT.stl scale=0.001 0.001 0.001; visual mesh filename=package://robot_description/meshes/WheelRT.stl scale=0.001 0.001 0.001
- added link base_link
- link camera_link: mass 0.1 -> 0.034782271109813245; geometry collision mesh filename=package://robot_description/meshes/Camera.stl scale=0.001 0.001 0.001; visual mesh filename=package://robot_description/meshes/Camera.stl scale=0.001 0.001 0.001
- link chassis: mass 5.0 -> 1.1414461681926555; geometry collision mesh filename=package://robot_description/meshes/Midsection.stl scale=0.001 0.001 0.001; visual mesh filename=package://robot_description/meshes/Midsection.stl scale=0.001 0.001 0.001
- link imu_link: mass None -> 0.001015546355999999; geometry collision mesh filename=package://robot_description/meshes/IMU.stl scale=0.001 0.001 0.001; visual mesh filename=package://robot_description/meshes/IMU.stl scale=0.001 0.001 0.001
- link left_wheel: mass 0.5 -> 0.03283332582192767; geometry collision mesh filename=package://robot_description/meshes/Drive-L.stl scale=0.001 0.001 0.001; visual mesh filename=package://robot_description/meshes/Drive-L.stl scale=0.001 0.001 0.001
- link lidar_link: mass 0.2 -> 0.04573956786244869; geometry collision mesh filename=package://robot_description/meshes/Lidar.stl scale=0.001 0.001 0.001; visual mesh filename=package://robot_description/meshes/Lidar.stl scale=0.001 0.001 0.001
- link right_wheel: mass 0.5 -> 0.03283328877308707; geometry collision mesh filename=package://robot_description/meshes/Drive-R.stl scale=0.001 0.001 0.001; visual mesh filename=package://robot_description/meshes/Drive-R.stl scale=0.001 0.001 0.001
Joints:
- removed joint camera_joint
- removed joint caster_joint
- removed joint imu_joint
- removed joint lidar_joint
- added joint Midsection_Revolute-55: type continuous, parent chassis, child WheelRT, origin xyz=0.22 0.0158 0.045 rpy=-1.5707963267948966 -0.0 0.0, axis 0.0 0.0 1.0
- added joint Midsection_Revolute-56: type fixed, parent chassis, child SLOTRBI, origin xyz=0.05649393 0.0158 0.044996299999999996 rpy=-1.5707963267948966 -0.0 0.0
- added joint Midsection_Revolute-57: type fixed, parent chassis, child SLOTRFI, origin xyz=0.1035 0.0158 0.045 rpy=-1.5707963267948966 -0.0 0.0
- added joint Midsection_Revolute-61: type continuous, parent chassis, child WheelLT, origin xyz=0.22 0.1672 0.045 rpy=1.5707963267948966 -0.0 0.0, axis 0.0 -3.19228529882681e-32 -1.0
- added joint Midsection_Revolute-62: type fixed, parent chassis, child SLOTLFI, origin xyz=0.1035 0.1672 0.045 rpy=1.5707963267948966 -0.0 0.0
- added joint Midsection_Revolute-63: type fixed, parent chassis, child SLOTLBI, origin xyz=0.05649393 0.1672 0.044996299999999996 rpy=1.5707963267948966 -0.0 0.0
- added joint Midsection_Rigid-66: type fixed, parent chassis, child MR, origin xyz=-0.06 0.044500000000000005 0.03825 rpy=1.5707963267948966 -0.0 0.0
- added joint Midsection_Rigid-67: type fixed, parent chassis, child ML, origin xyz=-0.06 0.1385 0.03825 rpy=1.5707963267948966 -0.0 0.0
- added joint Midsection_Rigid-68: type fixed, parent chassis, child Stepper-1, origin xyz=0.07864322 0.09150000000000001 0.05855968 rpy=3.141592653589793 -0.0 0.0
- added joint Midsection_Rigid-69: type fixed, parent chassis, child camera_link, origin xyz=0.219 0.0915 0.045 rpy=0.0 0.0 0.0
- added joint Midsection_Rigid-70: type fixed, parent chassis, child imu_link, origin xyz=0.21356999969482422 0.0915 0.07157500076293945 rpy=0.0 0.0 0.0
- added joint Midsection_Rigid-71: type fixed, parent chassis, child lidar_link, origin xyz=0.2135050018310547 0.0915 0.09840000152587891 rpy=0.0 0.0 0.0
- added joint Midsection_Rigid-72: type fixed, parent chassis, child Unyaktig-batteri-mockup-v1, origin xyz=-0.1085 0.1385 0.07575 rpy=-1.393221043589796e-15 -1.5707963267948966 0
- added joint SLOTLBI_Revolute-65: type continuous, parent SLOTLBI, child WheelLB, origin xyz=-0.07649393 -0.044996299999999996 0.0 rpy=4.26353305598774e-31 -5.9636863764438586e-161 -1.903778834633546e-192, axis -5.9636863764438586e-161 -3.944304526105059e-31 -1.0
- added joint SLOTLFI_Revolute-64: type continuous, parent SLOTLFI, child WheelLF, origin xyz=0.07651517000000001 -0.04496365 0.0 rpy=4.26353305598774e-31 -5.9636863764438586e-161 -1.903778834633546e-192, axis -5.9636863764438586e-161 -3.944304526105059e-31 -1.0
- added joint SLOTRBI_Revolute-58: type continuous, parent SLOTRBI, child WheelRB, origin xyz=-0.07649393 0.044996299999999996 0.0 rpy=-3.944304526105059e-31 5.9636863764438586e-161 0.0, axis -5.9636863764438586e-161 -3.944304526105059e-31 1.0
- added joint SLOTRFI_Revolute-59: type continuous, parent SLOTRFI, child WheelRF, origin xyz=0.07651517000000001 0.04496365 0.0 rpy=-3.944304526105059e-31 5.9636863764438586e-161 0.0, axis -5.9636863764438586e-161 -3.944304526105059e-31 1.0
- added joint chassis_to_base_link: type fixed, parent base_link, child chassis, origin xyz=-0.06325 -0.0915 0.023066925048828266 rpy=0.0 0.0 0.0
- joint left_wheel_joint: axis 0 0 1 -> 0.0 0.0 1.0; origin xyz=-0.035 0.093 -0.02 rpy=-1.5708 0 0 -> xyz=-0.06 0.16469999999999999 0.045250000000000005 rpy=-1.5707963267948966 -0.0 0.0
- joint right_wheel_joint: axis 0 0 1 -> 0.0 -3.081487911019579e-33 1.0; origin xyz=-0.035 -0.093 -0.02 rpy=-1.5708 0 0 -> xyz=-0.06 0.0183 0.045250000000000005 rpy=-1.5707963267948966 -0.0 0.0

Commit message: SIM med tracks og modell

File: src/robot_description/urdf/tracked_robot.urdf (robot description, URDF)
Before this commit: robot tracked_robot, 21 links, 20 joints
Links:
- added link left_track_rviz; visual box size=0.21 0.03 0.001; visual box size=0.21 0.03 0.007
- added link right_track_rviz; visual box size=0.21 0.03 0.001; visual box size=0.21 0.03 0.007
Joints:
- added joint left_track_rviz_joint: type fixed, parent chassis, child left_track_rviz, origin xyz=0.080 0.1835 -0.030 rpy=0 0 0
- added joint right_track_rviz_joint: type fixed, parent chassis, child right_track_rviz, origin xyz=0.080 -0.0005 -0.030 rpy=0 0 0
