Commit message: robot_description: new Fusion export (URDF, SDF, meshes)

File: src/robot_description/urdf/tracked_robot.urdf (robot description, URDF)
Before this commit: robot tracked_robot, 29 links, 28 joints
Links:
- removed link ML
- removed link MR
- removed link Robotarm
- removed link SLOTLBI
- removed link SLOTLFI
- removed link SLOTRBI
- removed link SLOTRFI
- removed link Stepper-1
- removed link Unyaktig-batteri-mockup-v1
- removed link WheelLB
- removed link WheelLF
- removed link WheelLT
- removed link WheelRB
- removed link WheelRF
- removed link WheelRT
- removed link chassis
- removed link gripper_plate
- removed link leadscrew
- removed link left_gripper_finger
- removed link left_track_rviz
- removed link left_wheel
- removed link right_gripper_finger
- removed link right_track_rviz
- removed link right_wheel
- removed link x_carriage
- added link ABX00102-Dist-sensor, mass 0.0016856916739247086; visual mesh filename=package://robot_description/meshes/ABX00102-Dist-sensor.stl scale=0.001 0.001 0.001
- added link BLLegs, mass 0.04732165189912416; visual mesh filename=package://robot_description/meshes/BLLegs.stl scale=0.001 0.001 0.001
- added link BN0085, mass 0.000971518679989001; visual mesh filename=package://robot_description/meshes/BN0085.stl scale=0.001 0.001 0.001
- added link BRLegs, mass 0.04732165189912416; visual mesh filename=package://robot_description/meshes/BRLegs.stl scale=0.001 0.001 0.001
- added link Bottom-Rack-200.0mm-L30.00-m2.1651, mass 0.02619004416035449; visual mesh filename=package://robot_description/meshes/Bottom-Rack-200.0mm-L30.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 scale=0.001 0.001 0.001
- added link Chassis, mass 1.4907690350907317; visual mesh filename=package://robot_description/meshes/Chassis.stl scale=0.001 0.001 0.001
- added link FLLegs, mass 0.04732234424542792; visual mesh filename=package://robot_description/meshes/FLLegs.stl scale=0.001 0.001 0.001
- added link FRLegs, mass 0.04732234424542792; visual mesh filename=package://robot_description/meshes/FRLegs.stl scale=0.001 0.001 0.001
- added link Finger-L-16L30.00-m2.1651, mass 0.04765014920834861; visual mesh filename=package://robot_description/meshes/Finger-L-16L30.00-m2.165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 scale=0.001 0.001 0.001
- added link Finger-R16L30.00-m2.1651Mirror, mass 0.047559344696753665; visual mesh filename=package://robot_description/meshes/Finger-R16L30.00-m2.1651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 scale=0.001 0.001 0.001
- added link Gear-9R24.00-m2.741-1-1, mass 0.01091885827041561; visual mesh filename=package://robot_description/meshes/Gear-9R24.00-m2.741-1-1.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 scale=0.001 0.001 0.001
- added link Gripper, mass 0.5425163222161179; visual mesh filename=package://robot_description/meshes/Gripper.stl scale=0.001 0.001 0.001
- added link LBWheel, mass 0.01930133239557942; visual mesh filename=package://robot_description/meshes/LBWheel.stl scale=0.001 0.001 0.001
- added link LBWheelColision, mass 0.4624031863395291; collision mesh filename=package://robot_description/meshes/LBWheelColision.stl scale=0.001 0.001 0.001; visual mesh filename=package://robot_description/meshes/LBWheelColision.stl scale=0.001 0.001 0.001
- added link LD06_LiDAR-1, mass 0.04311038533159423; visual mesh filename=package://robot_description/meshes/LD06_LiDAR-1.stl scale=0.001 0.001 0.001
- added link LDriveWheel, mass 0.03296579662050264; visual mesh filename=package://robot_description/meshes/LDriveWheel.stl scale=0.001 0.001 0.001
- added link LFWheel, mass 0.01930133239557942; visual mesh filename=package://robot_description/meshes/LFWheel.stl scale=0.001 0.001 0.001
- added link LLeadscrew, mass 0.3143219998584353; visual mesh filename=package://robot_description/meshes/LLeadscrew.stl scale=0.001 0.001 0.001
- added link LTWheel, mass 0.01930133239557942; visual mesh filename=package://robot_description/meshes/LTWheel.stl scale=0.001 0.001 0.001
- added link LTracks, mass 0.12017843301436808; collision box size=0.030 0.210 0.007; visual box size=0.030 0.210 0.007
- added link LeadNutL, mass 0.03449007966719112; visual mesh filename=package://robot_description/meshes/LeadNutL.stl scale=0.001 0.001 0.001
- added link LeadNutR, mass 0.03449007966719112; visual mesh filename=package://robot_description/meshes/LeadNutR.stl scale=0.001 0.001 0.001
- added link Leadscrew-Rigg, mass 0.2552161680137732; visual mesh filename=package://robot_description/meshes/Leadscrew-Rigg.stl scale=0.001 0.001 0.001
- added link M1, mass 0.17887898702311664; visual mesh filename=package://robot_description/meshes/M1.stl scale=0.001 0.001 0.001
- added link M2, mass 0.17887898702311664; visual mesh filename=package://robot_description/meshes/M2.stl scale=0.001 0.001 0.001
- added link Mega-wsheeld-v5-1, mass 0.11143362473176022; visual mesh filename=package://robot_description/meshes/Mega-wsheeld-v5-1.stl scale=0.001 0.001 0.001
- added link PI5, mass 0.01309093635557877; visual mesh filename=package://robot_description/meshes/PI5.stl scale=0.001 0.001 0.001
- added link RBWheel, mass 0.019302617704593204; visual mesh filename=package://robot_description/meshes/RBWheel.stl scale=0.001 0.001 0.001
- added link RBWheelColision, mass 0.4624031863395291; collision mesh filename=package://robot_description/meshes/RBWheelColision.stl scale=0.001 0.001 0.001; visual mesh filename=package://robot_description/meshes/RBWheelColision.stl scale=0.001 0.001 0.001
- added link RDriveWheel, mass 0.03296508821145091; visual mesh filename=package://robot_description/meshes/RDriveWheel.stl scale=0.001 0.001 0.001
- added link RFWheel, mass 0.01930261770459319; visual mesh filename=package://robot_description/meshes/RFWheel.stl scale=0.001 0.001 0.001
- added link RFWheelColision, mass 0.4624031863395291; collision mesh filename=package://robot_description/meshes/RFWheelColision.stl scale=0.001 0.001 0.001; visual mesh filename=package://robot_description/meshes/RFWheelColision.stl scale=0.001 0.001 0.001
- added link RFWheelColision-1, mass 0.4624031863395291; collision mesh filename=package://robot_description/meshes/RFWheelColision-1.stl scale=0.001 0.001 0.001; visual mesh filename=package://robot_description/meshes/RFWheelColision-1.stl scale=0.001 0.001 0.001
- added link RLeadscrew, mass 0.31432199985843523; visual mesh filename=package://robot_description/meshes/RLeadscrew.stl scale=0.001 0.001 0.001
- added link RTWheel, mass 0.01930261770459319; visual mesh filename=package://robot_description/meshes/RTWheel.stl scale=0.001 0.001 0.001
- added link RTracks, mass 0.12017843301436808; collision box size=0.030 0.210 0.007; visual box size=0.030 0.210 0.007
- added link Servo, mass 0.08417757927421474; visual mesh filename=package://robot_description/meshes/Servo.stl scale=0.001 0.001 0.001
- added link Servo-Gear-8L30.00-m2.1651, mass 0.002870206785412932; visual mesh filename=package://robot_description/meshes/Servo-Gear-8L30.00-m2.16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 scale=0.001 0.001 0.001
- added link Stepper-Gear-9R24.00-m2.741-1, mass 0.011184599309797512; visual mesh filename=package://robot_description/meshes/Stepper-Gear-9R24.00-m2.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 scale=0.001 0.001 0.001
- added link StøtteStag-1, mass 0.06992645940152016; visual mesh filename=package://robot_description/meshes/StøtteStag-1.stl scale=0.001 0.001 0.001
- added link Top-Rack-200.0mm-R30.00-m2.1651, mass 0.02617962275433629; visual mesh filename=package://robot_description/meshes/Top-Rack-200.0mm-R30.00-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 scale=0.001 0.001 0.001
- added link Unyaktig-batteri-mockup-v1-1, mass 0.44056121916666674; visual mesh filename=package://robot_description/meshes/Unyaktig-batteri-mockup-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 scale=0.001 0.001 0.001
- added link Xstepper, mass 0.4621945983755269; visual mesh filename=package://robot_description/meshes/Xstepper.stl scale=0.001 0.001 0.001
- added link ZStepper, mass 0.24015056879172078; visual mesh filename=package://robot_description/meshes/ZStepper.stl scale=0.001 0.001 0.001
- added link rps-kamera-v2-2, mass 0.003595639137613823; visual mesh filename=package://robot_description/meshes/rps-kamera-v2-2.stl scale=0.001 0.001 0.001
- link camera_link: mass 0.034782271109813245 -> None; geometry 
- link imu_link: mass 0.001015546355999999 -> None; geometry 
- link lidar_link: mass 0.04573956786244869 -> None; geometry 
Joints:
- removed joint Midsection_Revolute-55
- removed joint Midsection_Revolute-56
- removed joint Midsection_Revolute-57
- removed joint Midsection_Revolute-61
- removed joint Midsection_Revolute-62
- removed joint Midsection_Revolute-63
- removed joint Midsection_Rigid-66
- removed joint Midsection_Rigid-67
- removed joint Midsection_Rigid-68
- removed joint Midsection_Rigid-69
- removed joint Midsection_Rigid-70
- removed joint Midsection_Rigid-71
- removed joint Midsection_Rigid-72
- removed joint SLOTLBI_Revolute-65
- removed joint SLOTLFI_Revolute-64
- removed joint SLOTRBI_Revolute-58
- removed joint SLOTRFI_Revolute-59
- removed joint chassis_to_base_link
- removed joint leadscrew_to_base_link
- removed joint left_track_rviz_joint
- removed joint left_wheel_joint
- removed joint plate_arm_link
- removed joint right_track_rviz_joint
- removed joint right_wheel_joint
- added joint BLLegs_Revolute-10: type fixed, parent BLLegs, child LBWheel, origin xyz=-0.01549999999999999 -0.05876532 0.06650282 rpy=1.5707963267948974 -3.8761492285297827e-31 1.570796326794897
- added joint BLLegs_Revolute-43: type continuous, parent BLLegs, child LBWheelColision, origin xyz=-0.01549999999999999 -0.05876532 0.06650282 rpy=1.5707963267948974 -3.8761492285297827e-31 1.570796326794897, axis -3.8064789415719646e-16 8.049125398861855e-16 1.0
- added joint BRLegs_Revolute-3: type fixed, parent BRLegs, child RBWheel, origin xyz=0.01549999999999999 0.05876532 -0.06650282 rpy=1.5707963267948974 -2.465190328815662e-31 -1.5707963267948961
- added joint BRLegs_Revolute-44: type continuous, parent BRLegs, child RBWheelColision, origin xyz=0.01549999999999999 0.05876532 -0.06650282 rpy=1.5707963267948974 -2.465190328815662e-31 -1.5707963267948961, axis 3.8064789415719646e-16 -8.049125398861855e-16 -1.0
- added joint Chassis_Revolute-1: type revolute, parent Chassis, child BRLegs, origin xyz=0.05649392620590695 0.01579999999999999 0.044996302057189935 rpy=-1.5707963267948961 3.8064789415719715e-16 -1.5707963267948974, axis -1.0 4.930380657631324e-32 -1.4489281932630845e-31, limit lower=0.0 upper=0.261799 effort=1000000 velocity=1000000
- added joint Chassis_Revolute-11: type fixed, parent Chassis, child LDriveWheel, origin xyz=-0.0600000037940929 0.16470000000000004 0.045250002057189945 rpy=1.570796326794897 3.8064789415719715e-16 -1.5707963267948974
- added joint Chassis_Revolute-12: type fixed, parent Chassis, child LTWheel, origin xyz=0.219999996205907 0.16719999999999982 0.04500000205719005 rpy=1.570796326794897 3.8064789415719715e-16 -1.5707963267948974
- added joint Chassis_Revolute-2: type revolute, parent Chassis, child FRLegs, origin xyz=0.10350000620590694 0.015799999999999956 0.04500000205718996 rpy=-1.5707963267948961 3.8064789415719715e-16 -1.5707963267948974, axis -1.0 4.930380657631324e-32 -1.4489281932630845e-31, limit lower=-0.261799 upper=0.0 effort=1000000 velocity=1000000
- added joint Chassis_Revolute-5: type fixed, parent Chassis, child RTWheel, origin xyz=0.2199999962059069 0.015799999999999866 0.04500000205718999 rpy=-1.5707963267948961 3.8064789415719715e-16 -1.5707963267948974
- added joint Chassis_Revolute-6: type fixed, parent Chassis, child RDriveWheel, origin xyz=-0.060000003794093 0.01830000000000009 0.04525000205718989 rpy=-1.5707963267948961 3.8064789415719715e-16 -1.5707963267948974
- added joint Chassis_Revolute-7: type revolute, parent Chassis, child FLLegs, origin xyz=0.10350000620590706 0.16719999999999988 0.04500000205719001 rpy=1.570796326794897 3.8064789415719715e-16 -1.5707963267948974, axis 1.0 4.930380657631324e-32 -1.4489281932630845e-31, limit lower=0.0 upper=0.261799 effort=1000000 velocity=1000000
- added joint Chassis_Revolute-8: type revolute, parent Chassis, child BLLegs, origin xyz=0.056493926205907076 0.16719999999999993 0.04499630205718999 rpy=1.570796326794897 3.8064789415719715e-16 -1.5707963267948974, axis 1.0 4.930380657631324e-32 -1.4489281932630845e-31, limit lower=-0.261799 upper=0.0 effort=1000000 velocity=1000000
- added joint Chassis_Rigid-13: type fixed, parent Chassis, child Mega-wsheeld-v5-1, origin xyz=-0.06407910379409298 0.04384028000000006 0.08771429205718988 rpy=3.1415926535897927 -0.0955254270423661 1.5707963267948957
- added joint Chassis_Rigid-14: type fixed, parent Chassis, child ZStepper, origin xyz=0.07864321620590699 0.09149999999999993 0.05855968205718996 rpy=3.806478941571966e-16 3.8064789415719715e-16 -1.5707963267948974
- added joint Chassis_Rigid-15: type fixed, parent Chassis, child PI5, origin xyz=0.191999996205907 0.13719999999999982 0.07175000205719004 rpy=3.806478941571966e-16 3.8064789415719715e-16 -1.5707963267948974
- added joint Chassis_Rigid-16: type fixed, parent Chassis, child LD06_LiDAR-1, origin xyz=0.23059999620590696 0.07739999999999982 0.08275000205719002 rpy=3.806478941571966e-16 3.8064789415719715e-16 -1.5707963267948974
- added joint Chassis_Rigid-17: type fixed, parent Chassis, child BN0085, origin xyz=0.22470999620590695 0.08133999999999983 0.07275000205719001 rpy=-3.1415926535897927 3.8064789415719715e-16 -1.5707963267948974
- added joint Chassis_Rigid-18: type fixed, parent Chassis, child rps-kamera-v2-2, origin xyz=0.21499999620590693 0.10189999999999982 0.06275000205719003 rpy=1.5707963267948957 -1.5707963267948961 0
- added joint Chassis_Rigid-19: type fixed, parent Chassis, child Unyaktig-batteri-mockup-v1-1, origin xyz=-0.1086300237940929 0.09150000000000011 0.006242222057189899 rpy=-1.5707963267948961 -1.989750355821705e-16 -2.419782393886413e-15
- added joint Chassis_Rigid-20: type fixed, parent Chassis, child RLeadscrew, origin xyz=0.129443206205907 0.06299999999999993 -0.0014403179428100232 rpy=-3.1415926535897927 3.8064789415719715e-16 -1.5707963267948974
- added joint Chassis_Rigid-21: type fixed, parent Chassis, child LLeadscrew, origin xyz=0.12944320620590702 0.11899999999999991 -0.001440317942810001 rpy=-3.1415926535897927 3.8064789415719715e-16 -1.5707963267948974
- added joint Chassis_Rigid-27: type fixed, parent Chassis, child StøtteStag-1, origin xyz=0.05794320620590703 0.12499999999999994 0.056559682057189975 rpy=-3.1415926535897927 3.8064789415719715e-16 -1.5707963267948974
- added joint Chassis_Rigid-37: type fixed, parent Chassis, child M1, origin xyz=-0.0600000037940929 0.16270000000000004 0.045250002057189945 rpy=1.570796326794897 3.8064789415719715e-16 -1.5707963267948974
- added joint Chassis_Rigid-38: type fixed, parent Chassis, child M2, origin xyz=-0.060000003794093 0.020300000000000092 0.04525000205718989 rpy=-1.5707963267948961 3.8064789415719715e-16 -1.5707963267948974
- added joint Chassis_Rigid-40: type fixed, parent Chassis, child LTracks, origin xyz=0.07999578620590705 0.16719999999999993 0.059998152057189995 rpy=3.806478953373988e-16 -7.874654083273897e-05 -1.5707963267948974
- added joint Chassis_Rigid-41: type fixed, parent Chassis, child RTracks, origin xyz=0.07999578620590693 0.015799999999999967 0.05999815205718994 rpy=3.806478953373988e-16 -7.874654083292792e-05 -1.5707963267948974
- added joint Chassis_to_camera_link: type fixed, parent Chassis, child camera_link, origin xyz=0.21499999620590693 0.10189999999999982 0.06275000205719003 rpy=0 0 0
- added joint Chassis_to_imu_link: type fixed, parent Chassis, child imu_link, origin xyz=0.22470999620590695 0.08133999999999983 0.07275000205719001 rpy=0 0 0
- added joint Chassis_to_lidar_link: type fixed, parent Chassis, child lidar_link, origin xyz=0.23059999620590696 0.07739999999999982 0.08275000205719002 rpy=0 0 0
- added joint FLLegs_Revolute-42: type continuous, parent FLLegs, child RFWheelColision-1, origin xyz=-0.01549999999999999 -0.05873733 -0.06652989999999999 rpy=-1.5707963267948957 -3.8761492285297827e-31 1.570796326794897, axis 3.8064789415719626e-16 8.049125398861859e-16 1.0
- added joint FLLegs_Revolute-9: type fixed, parent FLLegs, child LFWheel, origin xyz=-0.01549999999999999 -0.05873733 -0.06652989999999999 rpy=1.5707963267948974 -3.8761492285297827e-31 1.570796326794897
- added joint FRLegs_Revolute-4: type fixed, parent FRLegs, child RFWheel, origin xyz=0.01549999999999999 0.05873733 0.06652989999999999 rpy=-1.5707963267948957 -2.465190328815662e-31 -1.5707963267948961
- added joint FRLegs_Revolute-45: type continuous, parent FRLegs, child RFWheelColision, origin xyz=0.01549999999999999 0.05873733 0.06652989999999999 rpy=1.5707963267948974 -2.465190328815662e-31 -1.5707963267948961, axis 3.8064789415719616e-16 -8.049125398861859e-16 -1.0
- added joint Gripper_Rigid-30: type fixed, parent Gripper, child Servo, origin xyz=-0.01075 0.15057500000000001 -0.15480967999999998 rpy=3.141592653589793 -1.5707963267948966 0
- added joint Gripper_Rigid-31: type fixed, parent Gripper, child ABX00102-Dist-sensor, origin xyz=0.0 0.185 -0.15391655999999998 rpy=-3.141592653589793 1.5707963267948966 0
- added joint Gripper_Slider-33: type fixed, parent Gripper, child Top-Rack-200.0mm-R30.00-m2.1651, origin xyz=-0.06508702 0.16570113000000003 -0.13650968 rpy=-3.141592653589793 -4.930380657631324e-32 -1.7755910601422187e-32
- added joint Gripper_Slider-34: type fixed, parent Gripper, child Bottom-Rack-200.0mm-L30.00-m2.1651, origin xyz=0.06492049 0.16570124 -0.17300967999999997 rpy=9.860761315262648e-32 -4.930380657631324e-32 -1.7755910601422187e-32
- added joint Leadscrew-Rigg_Revolute-26: type fixed, parent Leadscrew-Rigg, child Stepper-Gear-9R24.00-m2.741-1, origin xyz=-0.028000000000000004 -0.046 -0.32900000000000007 rpy=1.5707963267948966 2.4651903288156628e-31 -1.6412823737069552e-31
- added joint Leadscrew-Rigg_Revolute-28: type fixed, parent Leadscrew-Rigg, child Gear-9R24.00-m2.741-1-1, origin xyz=-0.028000000000000004 0.024000000000000004 -0.32900000000000007 rpy=1.5707963267948966 2.4651903288156628e-31 -1.6412823737069552e-31
- added joint Leadscrew-Rigg_Rigid-23: type fixed, parent Leadscrew-Rigg, child LeadNutR, origin xyz=0.0 0.0 -0.3525 rpy=3.141592653589793 9.860761315262648e-32 -3.6134346367594863e-31
- added joint Leadscrew-Rigg_Rigid-25: type fixed, parent Leadscrew-Rigg, child Xstepper, origin xyz=-0.043 -0.046 -0.32900000000000007 rpy=1.5707963267948966 9.860761315262648e-32 -9.736333669843527e-32
- added joint Leadscrew-Rigg_Rigid-39: type fixed, parent Leadscrew-Rigg, child LeadNutL, origin xyz=-0.055999999999999994 0.0 -0.3525 rpy=-3.141592653589793 -2.9605947323337477e-16 -3.6891410794762184e-31
- added joint Servo_Revolute-32: type fixed, parent Servo, child Servo-Gear-8L30.00-m2.1651, origin xyz=-8.881784197001253e-18 -0.01620000000000001 0.010749999999999989 rpy=1.5707963267948966 -1.5707963267948966 0
- added joint base_link_to_Chassis: type fixed, parent base_link, child Chassis, origin xyz=-0.06325 -0.0915 0.03998292504882827 rpy=0 0 0
- joint left_gripper_finger_joint: axis 0 0 1 -> 4.930380657631324e-32 4.930380657631326e-32 1.0000000000000007; child left_gripper_finger -> Finger-L-16L30.00-m2.1651; limit lower=-0.785 upper=0.785 effort=10 velocity=1.0 -> lower=-3.228859 upper=-0.523599 effort=1000000 velocity=1000000; origin xyz=0.0 0.0625 0.0 rpy=0 0 0 -> xyz=-0.05 0.19514971000000003 -0.15470968 rpy=-3.141592653589793 -5.473822126268811e-47 -2.0088433502773093e-31; parent gripper_plate -> Gripper
- joint right_gripper_finger_joint: axis 0 0 1 -> 4.930380657631324e-32 4.930380657631326e-32 1.0000000000000007; child right_gripper_finger -> Finger-R16L30.00-m2.1651Mirror; limit lower=-0.785 upper=0.785 effort=10 velocity=1.0 -> lower=0.523599 upper=2.96706 effort=1000000 velocity=1000000; origin xyz=0.0 -0.0625 0.0 rpy=0 0 0 -> xyz=0.05 0.19514971000000003 -0.15470968 rpy=-3.141592653589793 -5.473822126268811e-47 -2.0088433502773093e-31; parent gripper_plate -> Gripper
- joint robotarm_x_joint: axis 1 0 0 -> -6.676490067226021e-32 1.0 0.0; child x_carriage -> Gripper; limit lower=-0.2 upper=0.2 effort=100 velocity=0.01 -> lower=0.01 upper=0.09 effort=1000000 velocity=1000000; origin xyz=0.05 0.0 0.05 rpy=0 0 0 -> xyz=-0.028000000000000004 -0.011000000000000006 -0.319 rpy=-9.860761315262648e-32 9.860761315262648e-32 -9.736333669843527e-32; parent base_link -> Leadscrew-Rigg
- joint robotarm_z_joint: axis 0 0 1 -> 4.930380657631324e-32 4.930380657631324e-32 1.0; child Robotarm -> Leadscrew-Rigg; limit lower=1.0 upper=1.0 effort=100 velocity=0.01 -> lower=0.0 upper=0.25 effort=1000000 velocity=1000000; origin xyz=0.0 0.0 0.0 rpy=0 0 0 -> xyz=0.0 0.0 -0.500259 rpy=-3.141592653589793 9.860761315262648e-32 -8.292084300511961e-32; parent x_carriage -> RLeadscrew

Commit message: robot: port to new Fusion export (Tank3), fix sideways driving
- New model.sdf built from Fusion Gazebo.sdf with:
  - base_link root (yaw=+pi/2 in model frame) for correct ROS forward axis
  - TrackedVehicle drive proxy boxes on LTracks/RTracks (fdir1=0 1 0)
  - Spring/damping on 4 suspension joints (Chassis_Revolute-1/2/7/8)
  - Camera, IMU, LiDAR sensors on Chassis link
  - All plugins: TrackedVehicle, TrackController x2, JointPositionController x4,
    JointStatePublisher, PosePublisher
- World spawn yaw set to -pi/2 to cancel base_link rotation:
  base_link world yaw=0, forward=base_link X=track fdir1 direction
- Mesh update: removed 21 obsolete STL files, updated all 45 new STL files
- URDF: updated base_link_to_Chassis origin to match new Fusion geometry
- Added scripts/build_model_sdf.py for reproducible model.sdf generation

File: src/robot_description/urdf/tracked_robot.urdf (robot description, URDF)
Before this commit: robot tracked_robot, 49 links, 48 joints
Joints:
- joint base_link_to_Chassis: origin xyz=-0.06325 -0.0915 0.03998292504882827 rpy=0 0 0 -> xyz=-0.06164321620590698 -0.09150000000000008 0.024978117942810095 rpy=0 0 0

Commit message: modified:   config/robotarm_sim_params.yaml 	modified:   src/mekk4_bringup/mekk4_bringup/robotarm_safety_node.py 	modified:   src/mekk4_bringup/mekk4_bringup/ros_keyboard_teleop.py 	modified:   src/robot_bringup/launch/minimal_all.launch.py 	modified:   src/robot_description/urdf/tracked_robot.urdf 	modified:   src/robot_gz/models/tracked_robot/model.sdf 	modified:   src/robot_sim_control/robot_sim_control/gripper_sim_adapter.py 	modified:   src/robot_sim_control/robot_sim_control/robotarm_gui.py

File: src/robot_description/urdf/tracked_robot.urdf (robot description, URDF)
Before this commit: robot tracked_robot, 49 links, 48 joints
Joints:
- joint left_gripper_finger_joint: limit lower=-3.228859 upper=-0.523599 effort=1000000 velocity=1000000 -> lower=0.0 upper=8.0 effort=1000000 velocity=1000000
- joint right_gripper_finger_joint: limit lower=0.523599 upper=2.96706 effort=1000000 velocity=1000000 -> lower=0.0 upper=8.0 effort=1000000 velocity=1000000
- joint robotarm_x_joint: limit lower=0.01 upper=0.09 effort=1000000 velocity=1000000 -> lower=-0.07 upper=0.082 effort=1000000 velocity=1000000
