Commit message: modified:   Makefile 	modified:   config/robotarm_params.yaml 	deleted:    config/robotarm_sim_params.yaml 	modified:   config/teddy_approach.yaml 	modified:   config/teddy_grab.yaml 	new file:   src/mekk4_bringup/mekk4_bringup/dist_sensor_marker_node.py 	modified:   src/mekk4_bringup/mekk4_bringup/robotarm_safety_node.py 	modified:   src/mekk4_bringup/mekk4_bringup/ros_keyboard_teleop.py 	modified:   src/mekk4_bringup/mekk4_bringup/teddy_approach_node.py 	modified:   src/mekk4_bringup/mekk4_bringup/teddy_grab_node.py 	modified:   src/mekk4_bringup/mekk4_bringup/teddy_lidar_markers_node.py 	modified:   src/mekk4_bringup/setup.py 	modified:   src/robot_bringup/CMakeLists.txt 	modified:   src/robot_bringup/launch/minimal_all.launch.py 	modified:   src/robot_bringup/launch/pi_robot.launch.py 	modified:   src/robot_bringup/rviz/rviz.rviz 	modified:   src/robot_description/urdf/tracked_robot.urdf 	modified:   src/robot_gz/models/sim_teddy_bear/model.sdf 	modified:   src/robot_gz/models/tracked_robot/model.sdf 	modified:   src/robot_gz/worlds/tracked_robot_world.sdf 	new file:   src/robot_sim_control/robot_sim_control/dist_sensor_bridge.py 	modified:   src/robot_sim_control/robot_sim_control/robotarm_gui.py 	new file:   src/robot_sim_control/robot_sim_control/robotarm_state_adapter.py 	modified:   src/robot_sim_control/setup.py

File: src/robot_description/urdf/tracked_robot.urdf (robot description, URDF)
Before this commit: robot tracked_robot, 49 links, 48 joints
Links:
- added link dist_sensor_link
Joints:
- added joint ABX00102_to_dist_sensor_link: type fixed, parent ABX00102-Dist-sensor, child dist_sensor_link, origin xyz=0 -0.001606 0 rpy=0 0 -1.5707963267948966
- joint Chassis_to_imu_link: origin xyz=0.22470999620590695 0.08133999999999983 0.07275000205719001 rpy=0 0 0 -> xyz=0.21582 0.09150 0.07357 rpy=0 0 -1.5707963267948966
- joint Chassis_to_lidar_link: origin xyz=0.23059999620590696 0.07739999999999982 0.08275000205719002 rpy=0 0 0 -> xyz=0.21649999620590696 0.09150000000000003 0.11105000205719002 rpy=0 0 0
